File: design/electrical/pcb-hmd-carrier-board/pcb-hmd-carrier-board2.kicad_pcb (KiCad board)
At the start: 6 copper layers, 145.5 x 49.6 mm, 312 parts, among them J1 SJ-43514-SMT-TR, J10 PROX SENSOR - SM05B-SURS-TF, J11 BM28B0.6-20DS/2-0.35V BUTTON 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, J2 BM28 BATTERY FLEX 5A + NTC/ID, J201 J_DISPLAY_LEFT 24586305010482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, J202 J_DISPLAY_RIGHT 2458630501048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, J301 Molex 503398-1892 (CM4 LITE O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, J6 TAG-CONNECT SERVICE PADS (NO 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, J7 DF40C-100DP-0.4V(51) TRACKING, J8 DX07S024JJ2R1300 ACCESSORY, J9 DX07S016JA1R1500 CHARGE/SERVI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, U1 TPS62825DMQR, U10 TLV75528PDBVR, U11 HD3SS3212IRKSR, U12 TPS25751DREFR, U13 CAT24C512WI-GT3, U14 UPD720202K8-711-BAA-A, U15 TLV803EA30DBZR, U16 TPS2553-1DRVR, U2 TPS568230RJER, U201 TC358870XBG(NOK) C3008712, U202 TC358870XBG(NOK) C3008712, U203 TLV62569DBVR, U204 TLV62569DBVR, U205 TLV62569DBVR, U206 TLV62569DBVR, U207 TPS65132B5YFFR, U208 MP3387AGRT-P, U209 PCA9306DCTR C123752, U210 TCA9539PWR 1V8 DISPLAY GPIO, U3 TLV320AIC3204IRHBR, U301 RT9742GGJ5 SD POWER (CM4 LITE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, U4 TPD4E05U06DQAR, U5 TUSB320LAIRWBR, U6 BQ25798RQMR, U7 TPD2EUSB30DRTR, U8 TPD4EUSB30DQAR, U9 TPD4EUSB30DQAR, Y1 24MHz, Y201 SIT8008ACE73-18E-48.000000E, Y202 SIT8008ACE73-18E-48.000000E

Commit message: Update routing
This is one of the last commit containing change on the pcb, we will focus on proper user facing ui change and system change to make the best platform before doing any other change on any pcb
Routing:
- net I2C_SDA: track 0.00 -> 180.9 mm, vias 0 -> 9
- net CHG_SDA: track 0.00 -> 80.1 mm, vias 0 -> 4
- net R_HPDI: track 0.00 -> 78.2 mm, vias 0 -> 4
- net I2S_LRCLK: track 0.00 -> 74.1 mm, vias 0 -> 3
- net AUDIO_MCLK: track 0.00 -> 67.5 mm, vias 0 -> 3
- net BT_ENABLE_N: track 0.00 -> 45.2 mm, vias 0 -> 3
- net L_1V15_CORE: track 0.00 -> 44.0 mm, vias 0 -> 4
- net WLED_FREQ: track 0.00 -> 41.7 mm, vias 0 -> 2
- net I2Ct_SCL: track 0.00 -> 40.8 mm, vias 0 -> 4
- net R_BIASDA: track 0.00 -> 37.1 mm, vias 0 -> 3
- net HDMI_R_DDC_SDA: track 0.00 -> 35.6 mm, vias 0 -> 3
- net BIAS_SW: track 0.00 -> 35.4 mm, vias 0 -> 2
- net TS: track 0.00 -> 34.9 mm, vias 0 -> 2
- net BIAS_FLY1: track 0.00 -> 33.9 mm, vias 0 -> 3
- net LCD_BIAS_ENP: track 0.00 -> 33.1 mm, vias 0 -> 4
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